File: GPSDOMonitor/hardware/GPSDOMonitor.sch (KiCad schematic (older format))
At the start: 0 parts

Commit message: Add 5.5v regulator schematic
Parts:
- added C1, C2: CBR04C409B5GAC, Capacitor_Ceramic:C_0402_1005Metric, symbol Capacitor_Ceramic:CBR04C409B5GAC
- added C3, C5: UMK105B7104KV-FR, Capacitor_Ceramic:C_0402_1005Metric, symbol Capacitor_Ceramic:UMK105B7104KV-FR
- added C4: UMK325AB7106KM-P, Capacitor_Ceramic:C_1210_3225Metric, symbol Capacitor_Ceramic:UMK325AB7106KM-P
- added C6: A768KE686M1GLAE038, Capacitor_Electrolytic:CP_Elec_KEMET_8mm, symbol Capacitor_Electrolytic:A768KE686M1GLAE038
- added J1: F31S-1A7L1-11050, Connector_Data:F31S-1A7L1-11050, symbol Connector_Data:F31S-1A7L1-11050
- added L1: 74437356047, Inductor:74437356047, symbol Inductor:74437356047
- added R1: CRGCQ0402F82K, Resistor:R_0402_1005Metric, symbol Resistor:CRGCQ0402F82K
- added R2: CRGCQ0402F10K, Resistor:R_0402_1005Metric, symbol Resistor:CRGCQ0402F10K
- added U1: PIC18LF2550-ISO, Package_SO:SOIC-28_Width7.50mm_Pitch1.27mm, symbol Microcontroller:PIC18LF2550-ISO
- added U2: TPS563231DRLR, Package_TO_SOT:SOT-563, symbol Power_Management:TPS563231DRLR
- added X1: ABM8W-20.0000MHZ-4-K1Z-T3, Crystal:Crystal_SMD_4Pin_3.2x2.5mm, symbol Crystal:ABM8W-20.0000MHZ-4-K1Z-T3
Connections:
- net labels added: +12V, +3V3, +5V5, 10MHz, GND, PP2S, UART2_RxD_HV, UART2_TxD_HV, UART3_RxD, UART3_TxD, UART4_TX
- wire segments 0 -> 110
Other:
- note added: "1"
- note added: "10"
- note added: "11"
- note added: "12"
- note added: "13"
- note added: "14"
- note added: "15"
- note added: "16"
- note added: "17"
- note added: "18"
- note added: "19"
- note added: "2"
- note added: "20"
- note added: "21"
- note added: "22"
- note added: "23"
- note added: "24"
- note added: "25"
- note added: "26"
- note added: "27"
- note added: "28"
- note added: "29"
- note added: "3"
- note added: "30"
- note added: "31"
- note added: "32"
- note added: "33"
- note added: "34"
- note added: "35"
- note added: "36"
- note added: "37"
- note added: "38"
- note added: "39"
- note added: "4"
- note added: "40"
- note added: "41"
- note added: "42"
- note added: "43"
- note added: "44"
- note added: "45"
- note added: "46"
- note added: "47"
- note added: "48"
- note added: "49"
- note added: "5"
- note added: "50"
- note added: "6"
- note added: "7"
- note added: "8"
- note added: "9"
- note added: "NOTE: The blue numbers are the\npin numbers on the GPSDO side."

Commit message: Add 3.3v regulator for main CPU logic
Parts:
- removed L1: 74437356047, Inductor:74437356047, symbol Inductor:74437356047
- added C10: EMK212BB7106KG-T, Capacitor_Ceramic:C_0805_2012Metric, symbol Capacitor_Ceramic:EMK212BB7106KG-T
- added C3, C8: UMK105B7104KV-FR, Capacitor_Ceramic:C_0402_1005Metric, symbol Capacitor_Ceramic:UMK105B7104KV-FR
- added C5: UMK325AB7106KM-P, Capacitor_Ceramic:C_1210_3225Metric, symbol Capacitor_Ceramic:UMK325AB7106KM-P
- added D1: SS14HE, Diode:SOD-323HE, symbol Diode:SS14HE
- added D2: 1N914BWT, Diode:SOD-523, symbol Diode:1N914BWT
- added L1: ASPI-7318-4R7M-T, Inductor:ASPI-7318, symbol Inductor:ASPI-7318-4R7M-T
- added L2: NR6028T150M, Inductor:NR6028, symbol Inductor:NR6028T150M
- added R3: CRGCQ0402F33K, Resistor:R_0402_1005Metric, symbol Resistor:CRGCQ0402F33K
- added R4: CRGCQ0402F10K, Resistor:R_0402_1005Metric, symbol Resistor:CRGCQ0402F10K
- added U2: MCP16301T-I_CHY, Package_TO_SOT:SOT-23-6, symbol Power_Management:MCP16301T-I_CHY
- J1: Actuator Color (none) -> Black; Actuator Material (none) -> Liquid Crystal Polymer (LCP), Glass Filled; Base Part Number (none) -> F31S-1A7L1; Cable End Type (none) -> Notched or Tabbed; Connector/Contact Type (none) -> Contacts, Vertical - 1 Sided; Contact Finish (none) -> Gold; Contact Finish Thickness (none) -> 1.97µin (0.050µm); Contact Material (none) -> Phosphor Bronze; Current Rating (Amps) (none) -> 0.5A; FFC, FCB Thickness (none) -> 0.30mm; Features (none) -> Solder Retention, Zero Insertion Force (ZIF); Flat Flex Type (none) -> FFC, FPC; Height Above Board (none) -> 0.228\" (5.80mm); Housing Color (none) -> Natural; Housing Material (none) -> Liquid Crystal Polymer (LCP), Glass Filled; Locking Feature (none) -> Flip Lock; Material Flammability Rating (none) -> UL94 V-0; Mating Cycles (none) -> 30; Mounting Type (none) -> Surface Mount; Number of Positions (none) -> 50; Operating Temperature (none) -> -40°C ~ 105°C; Packaging (none) -> Cut Tape (CT); Pitch (none) -> 0.020\" (0.50mm); Series (none) -> Aorora F31S; Termination (none) -> Solder; Voltage Rating (none) -> 50V
- renumbered C3 to C2, C2 to C6, C5 to C7, C6 to C9, U2 to U1, U1 to U3
Connections:
- wire segments 110 -> 145
Other:
- note added: "3.3v regulator"
- note added: "5.5v 3A regulator"

Commit message: Add shift registers for indication
Parts:
- added D3, D4, D5, D6, D7, D8, D9: 5977703607F, LED:5977703607F, symbol LED:5977703607F
- added Q1: MMBT3904LT1G, Package_TO_SOT:SOT-23, symbol Transistor_BJT:MMBT3904LT1G
- added R5: CRGCQ0402F1K0, Resistor:R_0402_1005Metric, symbol Resistor:CRGCQ0402F1K0
- added U4, U5: SN74HC595BRWNR, Package_DFN_QFN:X1QFN-16_EP_2.5x2.5mm, symbol Logic:SN74HC595BRWNR
- renumbered C6 to C4, C4 to C5, C5 to C6
Connections:
- net labels added: LED_PWM, OE, RCLK, SER, SRCLK
- wire segments 145 -> 223
Other:
- moved on the sheet: J1

Commit message: Route power supplies
Parts:
- added R1: CRG0402ZR, Resistor:R_0402_1005Metric, symbol Resistor:CRG0402ZR
- renumbered R1 to R2, R2 to R3, R3 to R4, R4 to R5, R5 to R6
Connections:
- wire segments 223 -> 224

Commit message: Route majority of the current board
Parts:
- added R10, R11, R12, R13, R14, R15, R16, R17, R18, R19, R20, R7, R8, R9: CRGCQ0402F68R, Resistor:R_0402_1005Metric, symbol Resistor:CRGCQ0402F68R
Connections:
- wire segments 224 -> 245
